Commit message: add: vpusher to the robot

File: asset/franka_panda_custom/panda_template.urdf (robot description, URDF)
Before this commit: robot panda, 9 links, 8 joints
Links:
- added link panda_grasptarget, mass 10; collision mesh filename=package://{v_pusher_name} scale=1 1 1; visual mesh filename=package://{v_pusher_name} scale=1 1 1
- added link panda_hand, mass .81; collision mesh filename=package://meshes/collision/hand.obj; visual mesh filename=package://meshes/visual/hand.obj
- added link panda_leftfinger, mass 0.1; collision mesh filename=package://meshes/collision/finger.obj; visual mesh filename=package://meshes/visual/finger.obj
- added link panda_rightfinger, mass 0.1; collision mesh filename=package://meshes/collision/finger.obj; visual mesh filename=package://meshes/visual/finger.obj
Joints:
- added joint panda_finger_joint1: type prismatic, parent panda_hand, child panda_leftfinger, origin xyz=0 0 0.0584 rpy=0 0 0, axis 0 1 0, limit lower=0.0 upper=0.04 effort=20 velocity=0.2
- added joint panda_finger_joint2: type prismatic, parent panda_hand, child panda_rightfinger, origin xyz=0 0 0.0584 rpy=0 0 0, axis 0 -1 0, limit lower=0.0 upper=0.04 effort=20 velocity=0.2, mimic joint=panda_finger_joint1
- added joint panda_grasptarget_hand: type fixed, parent panda_hand, child panda_grasptarget, origin xyz=0 0 0.100 rpy=0 0 0
- added joint panda_hand_joint: type fixed, parent panda_link8, child panda_hand, origin xyz=0 0 0 rpy=0 0 -0.785398163397

Commit message: fix: invisible panda after couple of resets - avoid loading arm each episode; load only vpusher

File: asset/franka_panda_custom/panda_template.urdf (robot description, URDF)
Before this commit: robot panda, 13 links, 12 joints
Links:
- removed link panda_grasptarget
Joints:
- removed joint panda_grasptarget_hand
