Commit message: add: dlr sim - env preparation

File: asset/lc_soft_enable_wide_grip/lc_soft_enable_wide_grip.urdf (robot description, URDF)
Before this commit: robot lc_soft_enable_wide_grip, 5 links, 4 joints
Links:
- link left_finger_link: geometry collision mesh filename=asset/lc_soft_enable_wide_grip/meshes/left_base_105.stl scale=0.001 0.001 0.001; visual mesh filename=asset/lc_soft_enable_wide_grip/meshes/left_base_105.stl scale=0.001 0.001 0.001
- link left_tip_link: geometry collision mesh filename=asset/lc_soft_enable_wide_grip/meshes/left_distal_45.stl scale=0.001 0.001 0.001; visual mesh filename=asset/lc_soft_enable_wide_grip/meshes/left_distal_45.stl scale=0.001 0.001 0.001
- link right_finger_link: geometry collision mesh filename=asset/lc_soft_enable_wide_grip/meshes/right_base_105.stl scale=0.001 0.001 0.001; visual mesh filename=asset/lc_soft_enable_wide_grip/meshes/right_base_105.stl scale=0.001 0.001 0.001
- link right_tip_link: geometry collision mesh filename=asset/lc_soft_enable_wide_grip/meshes/right_distal_45.stl scale=0.001 0.001 0.001; visual mesh filename=asset/lc_soft_enable_wide_grip/meshes/right_distal_45.stl scale=0.001 0.001 0.001
Joints:
- joint left_tip: origin xyz=0.0695 0.0 0.005375 rpy=-1.5707963267948968 0.8726640421845309 3.141592653589793 -> xyz=0.1145 0.0 0.005375 rpy=-1.5707963267948968 0.8726640421845309 3.141592653589793
- joint right_tip: origin xyz=0.0695 0.0 0.005375 rpy=-1.5707963267948963 0.87266404218453 3.141592653589793 -> xyz=0.1145 0.0 0.005375 rpy=-1.5707963267948963 0.87266404218453 3.141592653589793

Commit message: dlr tip curvature added

File: asset/lc_soft_enable_wide_grip/lc_soft_enable_wide_grip.urdf (robot description, URDF)
Before this commit: robot lc_soft_enable_wide_grip, 5 links, 4 joints
Links:
- removed link left_finger_link
- added link left_finger, mass 0.19324581; collision mesh filename=asset/lc_soft_enable_wide_grip/meshes/lc_soft_enable_wide_g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 scale=1.0 1.0 1.0; visual mesh filename=asset/lc_soft_enable_wide_grip/meshes/lc_soft_enable_wide_g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 scale=1.0 1.0 1.0
- link base_link: mass 1.088118 -> 0.98136109; geometry collision mesh filename=asset/lc_soft_enable_wide_grip/meshes/lc_soft_enable_wide_g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 scale=1.0 1.0 1.0; visual mesh filename=asset/lc_soft_enable_wide_grip/meshes/lc_soft_enable_wide_g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 scale=1.0 1.0 1.0
- link left_tip_link: mass 0.013727707 -> 0.01222309; geometry collision mesh filename=asset/lc_soft_enable_wide_grip/meshes/left_distal_50_6.stl scale=0.001 0.001 0.001; visual mesh filename=asset/lc_soft_enable_wide_grip/meshes/left_distal_50_6.stl scale=0.001 0.001 0.001
- link right_finger_link: mass 0.071622239 -> 0.19324581; geometry collision mesh filename=asset/lc_soft_enable_wide_grip/meshes/lc_soft_enable_wide_g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 scale=1.0 1.0 1.0; visual mesh filename=asset/lc_soft_enable_wide_grip/meshes/lc_soft_enable_wide_g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 scale=1.0 1.0 1.0
- link right_tip_link: mass 0.013727707 -> 0.01222309; geometry collision mesh filename=asset/lc_soft_enable_wide_grip/meshes/right_distal_50_6.stl scale=0.001 0.001 0.001; visual mesh filename=asset/lc_soft_enable_wide_grip/meshes/right_distal_50_6.stl scale=0.001 0.001 0.001
Joints:
- joint left_base: child left_finger_link -> left_finger; limit lower=0 upper=0.0575 effort=100 velocity=2 -> lower=0 upper=0.0575 effort=100000000000000000 velocity=100000000000000000; origin xyz=0.06658 4.689172593935216e-18 0.1335 rpy=1.874699728327322e-33 -1.5707963057214722 0 -> xyz=0.07658 4.689172593935216e-18 0.1335 rpy=1.874699728327322e-33 -1.5707963057214722 0
- joint left_tip: limit lower=0 upper=1.0471975511965976 effort=100 velocity=2 -> lower=0 upper=1.74 effort=100000000000000000 velocity=100000000000000000; origin xyz=0.1145 0.0 0.005375 rpy=-1.5707963267948968 0.8726640421845309 3.141592653589793 -> xyz=0.0715 4.727136644708785e-19 -0.00772 rpy=1.5707963267948966 2.220446049250313e-16 -1.2246467991473532e-16; parent left_finger_link -> left_finger
- joint right_finger: limit lower=0 upper=0.0575 effort=100 velocity=2 -> lower=0 upper=0.0575 effort=100000000000000000 velocity=100000000000000000; origin xyz=-0.06658 -4.689172593935216e-18 0.1335 rpy=-3.141592653589793 -1.5707963057214722 0 -> xyz=-0.07658 -4.689172593935216e-18 0.1335 rpy=-3.141592653589793 -1.5707963057214722 0
- joint right_tip: limit lower=0 upper=1.0471975511965976 effort=100 velocity=2 -> lower=-0.17 upper=1.74 effort=100000000000000000 velocity=100000000000000000; origin xyz=0.1145 0.0 0.005375 rpy=-1.5707963267948963 0.87266404218453 3.141592653589793 -> xyz=0.0715 -4.727136644708785e-19 -0.00772 rpy=1.5707963267948966 2.220446049250313e-16 -1.2246467991473535e-16
